Commit message: feat: try fitting real data and highlevel output

File: legged_gym/resources/robots/go1g/urdf/go1_gripper.urdf (robot description, URDF)
Before this commit: robot go1_description, 41 links, 40 joints
Links:
- added link gripper_grasp_point_link; collision empty ; visual sphere radius=0.001
Joints:
- added joint gripper_grasp_point_joint: type fixed, parent gripper_link, child gripper_grasp_point_link, origin xyz=0.15 0.0 -0.225 rpy=0 0 0, axis 0 -1 0, limit lower=0. upper=0.0

Commit message: feat: train pickup

File: legged_gym/resources/robots/go1g/urdf/go1_gripper.urdf (robot description, URDF)
Before this commit: robot go1_description, 42 links, 41 joints
Joints:
- joint l_finger_joint: limit lower=-0.04 upper=0.0 -> lower=-0.015 upper=-0.001 effort=1
- joint r_finger_joint: limit lower=-0.04 upper=0.0 -> lower=-0.015 upper=-0.001 effort=1; mimic joint=l_finger_joint multiplier=1 offset=0 -> (none)

Commit message: feat: use go2 now

File: legged_gym/resources/robots/go1g/urdf/go1_gripper.urdf (robot description, URDF)
Before this commit: robot go1_description, 42 links, 41 joints
Links:
- link l_finger_link: geometry collision box size=0.04 0.064 0.08; visual box size=0.04 0.064 0.08
- link r_finger_link: geometry collision box size=0.04 0.064 0.08; visual box size=0.04 0.064 0.08
Joints:
- joint l_finger_joint: limit lower=-0.015 upper=-0.001 effort=1 -> lower=-0.025 upper=-0.001 effort=10
- joint r_finger_joint: limit lower=-0.015 upper=-0.001 effort=1 -> lower=-0.025 upper=-0.001 effort=10
