Commit message: feat: check between fingers

File: legged_gym/resources/robots/go2/urdf/go2g_description_v5.urdf (robot description, URDF)
Before this commit: robot go2g_description, 33 links, 32 joints
Links:
- link l_finger_link: geometry collision box size=0.04 0.12 0.16; visual box size=0.04 0.12 0.16
- link r_finger_link: geometry collision box size=0.04 0.12 0.16; visual box size=0.04 0.12 0.16
Joints:
- joint l_finger_joint: origin xyz=0.12 0.026 -0.13 rpy=0 0.523598 0 -> xyz=0.08 0.026 -0.25 rpy=0 -0.523598 0
- joint r_finger_joint: origin xyz=0.12 -0.026 -0.13 rpy=0 0.523598 0 -> xyz=0.08 -0.026 -0.25 rpy=0 -0.523598 0
