Commit message: train without fit or collision

File: legged_gym/resources/robots/go2/urdf/go2g_description_v4.urdf (robot description, URDF)
Before this commit: robot go2g_description, 33 links, 32 joints
Links:
- link l_finger_link: geometry collision box size=0.04 0.064 0.08; visual box size=0.04 0.064 0.08
- link r_finger_link: geometry collision box size=0.04 0.064 0.08; visual box size=0.04 0.064 0.08

Commit message: larger gripper collision

File: legged_gym/resources/robots/go2/urdf/go2g_description_v4.urdf (robot description, URDF)
Before this commit: robot go2g_description, 33 links, 32 joints
Links:
- link Head_lower: geometry collision sphere radius=0.0047
- link l_finger_link: geometry collision box size=0.02 0.12 0.16; visual mesh filename=../dae/finger.stl scale=0.001 0.001 0.001
- link r_finger_link: geometry collision box size=0.02 0.12 0.16; visual mesh filename=../dae/finger.stl scale=0.001 0.001 0.001

Commit message: feat: resample only in reset, larger gripper

File: legged_gym/resources/robots/go2/urdf/go2g_description_v4.urdf (robot description, URDF)
Before this commit: robot go2g_description, 33 links, 32 joints
Links:
- link l_finger_link: geometry collision box size=0.02 0.12 0.16; visual mesh filename=../dae/finger.stl scale=0.001 0.001 0.001
- link r_finger_link: geometry collision box size=0.02 0.12 0.16; visual mesh filename=../dae/finger.stl scale=0.001 0.001 0.001

Commit message: feat: add collision termination

File: legged_gym/resources/robots/go2/urdf/go2g_description_v4.urdf (robot description, URDF)
Before this commit: robot go2g_description, 33 links, 32 joints
Links:
- link Head_lower: geometry collision sphere radius=0.0047
Joints:
- joint gripper_grasp_point_joint: origin xyz=0.15 0.0 -0.225 rpy=0 0 0 -> xyz=0.19 0.0 -0.28 rpy=0 0 0

Commit message: feat: add termination after contact

File: legged_gym/resources/robots/go2/urdf/go2g_description_v4.urdf (robot description, URDF)
Before this commit: robot go2g_description, 33 links, 32 joints
Joints:
- joint gripper_grasp_point_joint: origin xyz=0.15 0.0 -0.225 rpy=0 0 0 -> xyz=0.19 0.0 -0.28 rpy=0 0 0

Commit message: feat: hold still; frac; ready_to_grasp

File: legged_gym/resources/robots/go2/urdf/go2g_description_v4.urdf (robot description, URDF)
Before this commit: robot go2g_description, 33 links, 32 joints
Links:
- link l_finger_link: geometry collision box size=0.03 0.064 0.08; visual mesh filename=../dae/finger.stl scale=0.001 0.001 0.001
- link r_finger_link: geometry collision box size=0.03 0.064 0.08; visual mesh filename=../dae/finger.stl scale=0.001 0.001 0.001
Joints:
- joint gripper_grasp_point_joint: origin xyz=0.19 0.0 -0.28 rpy=0 0 0 -> xyz=0.16 0.0 -0.26 rpy=0 0 0
- joint l_finger_joint: limit lower=-0.04 upper=0.0 -> lower=-0.04 upper=0.0 effort=10
- joint r_finger_joint: limit lower=-0.04 upper=0.0 -> lower=-0.04 upper=0.0 effort=10

Commit message: train

File: legged_gym/resources/robots/go2/urdf/go2g_description_v4.urdf (robot description, URDF)
Before this commit: robot go2g_description, 33 links, 32 joints
Links:
- link gripper_grasp_point_link: geometry 
- link l_finger_link: geometry collision box size=0.03 0.064 0.08; visual box size=0.03 0.064 0.08
- link r_finger_link: geometry collision box size=0.03 0.064 0.08; visual box size=0.03 0.064 0.08
